File: base.sch (EAGLE design)
At the start: 3 parts, among them J1 AS0A626-U2SN-7F, U2 XC7K160TFBG676

Commit message: updates, wired 33 + 34
Parts:
- removed U2: XC7K160TFBG676, xilinx_devices_V6:XC7K160TFBG676
- added B1: 1.5V seiko TS518FE_FL35E, battery:CH291-1220LF
- added C1, C2: .1uF, eagle-ltspice:CC0402
- added C157, C158, C163: 100UF, eagle-ltspice:CC1206
- added C461, C462, C490, C491: 0.1UF, eagle-ltspice:CC0402
- added D6: BAS40-04, diode:BAS40-04
- added DS10: (no value), led:LEDCHIP-LED0603
- added J52: (no value), pinhead:PINHD-1X2
- added R337, R338, R339: 1.21K, eagle-ltspice:RR0402
- added R396: 261, eagle-ltspice:RR0402
- added R83: 4.7K, eagle-ltspice:RR0402
- added SW1: SWS003, smd-special:SWS003
- added TP1, TP2: TP2P2-38-17, testpad:TP2P2-38-17
- added U1: XC7A200TFBG676, xilinx_devices_V6_custom_labels:XC7A200TFBG676
Connections:
- removed net D_A0: J1.98
- removed net D_A1: J1.97
- removed net D_A10: J1.107
- removed net D_A11: J1.84
- removed net D_A12: J1.83
- removed net D_A13: J1.119
- removed net D_A14: J1.80
- removed net D_A15: J1.78
- removed net D_A2: J1.96
- removed net D_A3: J1.95
- removed net D_A4: J1.92
- removed net D_A5: J1.91
- removed net D_A6: J1.90
- removed net D_A7: J1.86
- removed net D_A8: J1.89
- removed net D_A9: J1.85
- removed net D_BA0: J1.109
- removed net D_BA1: J1.108
- removed net D_BA2: J1.79
- removed net D_CAS_N: J1.115
- removed net D_CKE0: J1.73
- removed net D_CLK0_N: J1.103
- removed net D_CLK0_P: J1.101
- removed net D_CLK1_N: J1.104
- removed net D_CLK1_P: J1.102
- removed net D_D0: J1.5
- removed net D_D1: J1.7
- removed net D_D10: J1.33
- removed net D_D11: J1.35
- removed net D_D12: J1.22
- removed net D_D13: J1.24
- removed net D_D14: J1.34
- removed net D_D15: J1.36
- removed net D_D16: J1.39
- removed net D_D17: J1.41
- removed net D_D18: J1.51
- removed net D_D19: J1.53
- removed net D_D2: J1.15
- removed net D_D20: J1.40
- removed net D_D21: J1.42
- removed net D_D22: J1.50
- removed net D_D23: J1.52
- removed net D_D24: J1.57
- removed net D_D25: J1.59
- removed net D_D26: J1.67
- removed net D_D27: J1.69
- removed net D_D28: J1.56
- removed net D_D29: J1.58
- removed net D_D3: J1.17
- removed net D_D30: J1.68
- removed net D_D31: J1.70
- removed net D_D32: J1.129
- removed net D_D33: J1.131
- removed net D_D34: J1.141
- removed net D_D35: J1.143
- removed net D_D36: J1.130
- removed net D_D37: J1.132
- removed net D_D38: J1.140
- removed net D_D39: J1.142
- removed net D_D4: J1.4
- removed net D_D40: J1.147
- removed net D_D41: J1.149
- removed net D_D42: J1.157
- removed net D_D43: J1.159
- removed net D_D44: J1.146
- removed net D_D45: J1.148
- removed net D_D46: J1.158
- removed net D_D47: J1.160
- removed net D_D48: J1.163
- removed net D_D49: J1.165
- removed net D_D5: J1.6
- removed net D_D50: J1.175
- removed net D_D51: J1.177
- removed net D_D52: J1.164
- removed net D_D53: J1.166
- removed net D_D54: J1.174
- removed net D_D55: J1.176
- removed net D_D56: J1.181
- removed net D_D57: J1.183
- removed net D_D58: J1.191
- removed net D_D59: J1.193
- removed net D_D6: J1.16
- removed net D_D60: J1.180
- removed net D_D61: J1.182
- removed net D_D62: J1.192
- removed net D_D63: J1.194
- removed net D_D7: J1.18
- removed net D_D8: J1.21
- removed net D_D9: J1.23
- removed net D_DM0: J1.11
- removed net D_DM1: J1.28
- removed net D_DM2: J1.46
- removed net D_DM3: J1.63
- removed net D_DM4: J1.136
- removed net D_DM5: J1.153
- removed net D_DM6: J1.170
- removed net D_DM7: J1.187
- removed net D_DQS0_N: J1.10
- removed net D_DQS0_P: J1.12
- removed net D_DQS1_N: J1.27
- removed net D_DQS1_P: J1.29
- removed net D_DQS2_N: J1.45
- removed net D_DQS2_P: J1.47
- removed net D_DQS3_N: J1.62
- removed net D_DQS3_P: J1.64
- removed net D_DQS4_N: J1.135
- removed net D_DQS4_P: J1.137
- removed net D_DQS5_N: J1.152
- removed net D_DQS5_P: J1.154
- removed net D_DQS6_N: J1.169
- removed net D_DQS6_P: J1.171
- removed net D_DQS7_N: J1.186
- removed net D_DQS7_P: J1.188
- removed net D_NC: J1.120, J1.121, J1.122, J1.125, J1.74, J1.77
- removed net D_ODT0: J1.116
- removed net D_RAS_N: J1.110
- removed net D_RESET_N: J1.30
- removed net D_S0_N: J1.114
- removed net D_SCL: J1.202
- removed net D_SDA: J1.200
- removed net D_VSS: J1.127, J1.128, J1.13, J1.133, J1.134, J1.138, J1.139, J1.14, J1.144, J1.145, J1.150, J1.151, J1.155, J1.156, J1.161, J1.162, J1.167, J1.168, J1.172, J1.173, J1.178, J1.179, J1.184, J1.185, J1.189, J1.19, J1.190, J1.195, J1.196, J1.2, J1.20, J1.25, J1.26, J1.3, J1.31, J1.32, J1.37, J1.38, J1.43, J1.44, J1.48, J1.49, J1.54, J1.55, J1.60, J1.61, J1.65, J1.66, J1.71, J1.72, J1.8, J1.9
- removed net D_WE_N: J1.113
- removed net F_CCLK: U2B0.CCLK_0
- removed net F_DONE: U2B0.DONE_0
- removed net F_INIT_N: U2B0.INIT_B_0
- removed net F_M0: U2B0.M0_0
- removed net F_M1: U2B0.M1_0
- removed net F_M2: U2B0.M2_0
- removed net F_PROG_N: U2B0.PROGRAM_B_0
- removed net F_TCK_BUF: U2B0.TCK_0
- removed net F_TDI_BUF: U2B0.TDI_0
- removed net F_TDO: U2B0.TDO_0
- removed net F_TMS_BUF: U2B0.TMS_0
- removed net F_VBATT: U2B0.VCCBATT_0
- removed net VADJ_F: U2B12.VCCO_12@0, U2B12.VCCO_12@1, U2B12.VCCO_12@2, U2B12.VCCO_12@3, U2B12.VCCO_12@4, U2B12.VCCO_12@5, U2B12.VCCO_12@6, U2B13.VCCO_13@0, U2B13.VCCO_13@1, U2B13.VCCO_13@2, U2B13.VCCO_13@3, U2B13.VCCO_13@4, U2B13.VCCO_13@5, U2B16.VCCO_16@0, U2B16.VCCO_16@1, U2B16.VCCO_16@2, U2B16.VCCO_16@3, U2B16.VCCO_16@4, U2B16.VCCO_16@5, U2B16.VCCO_16@6
- removed net VCC1V5_F: U2B32.VCCO_32@0, U2B32.VCCO_32@1, U2B32.VCCO_32@2, U2B32.VCCO_32@3, U2B32.VCCO_32@4, U2B32.VCCO_32@5, U2B33.VCCO_33@0, U2B33.VCCO_33@1, U2B33.VCCO_33@2, U2B33.VCCO_33@3, U2B33.VCCO_33@4, U2B33.VCCO_33@5, U2B34.VCCO_34@0, U2B34.VCCO_34@1, U2B34.VCCO_34@2, U2B34.VCCO_34@3, U2B34.VCCO_34@4, U2B34.VCCO_34@5
- removed net VCC1V5_FPGA: J1.100, J1.105, J1.106, J1.111, J1.112, J1.117, J1.118, J1.123, J1.75, J1.76, J1.81, J1.82, J1.87, J1.88, J1.93, J1.94, J1.99
- removed net VCC2V5_F: U2B0.CFGBVS_0, U2B0.VCCO_0@0, U2B0.VCCO_0@1, U2B14.VCCO_14@0, U2B14.VCCO_14@1, U2B14.VCCO_14@2, U2B14.VCCO_14@3, U2B14.VCCO_14@4, U2B14.VCCO_14@5, U2B15.VCCO_15@0, U2B15.VCCO_15@1, U2B15.VCCO_15@2, U2B15.VCCO_15@3, U2B15.VCCO_15@4, U2B15.VCCO_15@5
- removed net VTTDDR: J1.203, J1.204
- new net CPU_RESET: U1B34.IO_25_34
- new net DDR3_28: U1B33.IO_L2N_T0_33
- new net DDR3_A0: U1B34.IO_L3P_T0_DQS_34
- new net DDR3_A1: U1B34.IO_L1N_T0_34
- new net DDR3_A10: U1B34.IO_L5P_T0_34
- new net DDR3_A11: U1B34.IO_L4P_T0_34
- new net DDR3_A12: U1B34.IO_L2N_T0_34
- new net DDR3_A13: U1B34.IO_L5N_T0_34
- new net DDR3_A14: U1B34.IO_L8P_T1_34
- new net DDR3_A15: U1B34.IO_L8N_T1_34
- new net DDR3_A2: U1B34.IO_L7N_T1_34
- new net DDR3_A3: U1B34.IO_L3N_T0_DQS_34
- new net DDR3_A4: U1B34.IO_L4N_T0_34
- new net DDR3_A5: U1B34.IO_L2P_T0_34
- new net DDR3_A6: U1B34.IO_L7P_T1_34
- new net DDR3_A7: U1B34.IO_L6P_T0_34
- new net DDR3_A8: U1B34.IO_L10N_T1_34
- new net DDR3_A9: U1B34.IO_L1P_T0_34
- new net DDR3_BA0: U1B34.IO_L9P_T1_DQS_34
- new net DDR3_BA1: U1B34.IO_L9N_T1_DQS_34
- new net DDR3_BA2: U1B34.IO_L10P_T1_34
- new net DDR3_CAS_B: U1B34.IO_L16P_T2_34
- new net DDR3_CKE0: U1B34.IO_L14P_T2_SRCC_34
- new net DDR3_CKE1: U1B34.IO_L14N_T2_SRCC_34
- new net DDR3_CLK0_N: U1B34.IO_L11N_T1_SRCC_34
- new net DDR3_CLK0_P: U1B34.IO_L11P_T1_SRCC_34
- new net DDR3_CLK1_N: U1B34.IO_L12N_T1_MRCC_34
- new net DDR3_CLK1_P: U1B34.IO_L12P_T1_MRCC_34
- new net DDR3_D0: U1B33.IO_L24P_T3_33
- new net DDR3_D1: U1B33.IO_L23N_T3_33
- new net DDR3_D10: U1B33.IO_L16N_T2_33
- new net DDR3_D11: U1B33.IO_L16P_T2_33
- new net DDR3_D12: U1B33.IO_L14N_T2_SRCC_33
- new net DDR3_D13: U1B33.IO_L14P_T2_SRCC_33
- new net DDR3_D14: U1B33.IO_L13N_T2_MRCC_33
- new net DDR3_D15: U1B33.IO_L13P_T2_MRCC_33
- new net DDR3_D16: U1B33.IO_L11N_T1_SRCC_33
- new net DDR3_D17: U1B33.IO_L11P_T1_SRCC_33
- new net DDR3_D18: U1B33.IO_L10N_T1_33
- new net DDR3_D19: U1B33.IO_L10P_T1_33
- new net DDR3_D2: U1B33.IO_L23P_T3_33
- new net DDR3_D20: U1B33.IO_L8N_T1_33
- new net DDR3_D21: U1B33.IO_L8P_T1_33
- new net DDR3_D22: U1B33.IO_L7N_T1_33
- new net DDR3_D23: U1B33.IO_L7P_T1_33
- new net DDR3_D24: U1B33.IO_L5N_T0_33
- new net DDR3_D25: U1B33.IO_L5P_T0_33
- new net DDR3_D26: U1B33.IO_L4N_T0_33
- new net DDR3_D27: U1B33.IO_L4P_T0_33
- new net DDR3_D29: U1B33.IO_L2P_T0_33
- new net DDR3_D3: U1B33.IO_L22N_T3_33
- new net DDR3_D30: U1B33.IO_L1N_T0_33
- new net DDR3_D31: U1B33.IO_L1P_T0_33
- new net DDR3_D4: U1B33.IO_L22P_T3_33
- new net DDR3_D5: U1B33.IO_L20N_T3_33
- new net DDR3_D6: U1B33.IO_L20P_T3_33
- new net DDR3_D7: U1B33.IO_L19P_T3_33
- new net DDR3_D8: U1B33.IO_L17N_T2_33
- new net DDR3_D9: U1B33.IO_L17P_T2_33
- new net DDR3_DM0: U1B33.IO_L24N_T3_33
- new net DDR3_DM1: U1B33.IO_L18P_T2_33
- new net DDR3_DM2: U1B33.IO_L12P_T1_MRCC_33
- new net DDR3_DM3: U1B33.IO_L6P_T0_33
- new net DDR3_DQS0_N: U1B33.IO_L21N_T3_DQS_33
- new net DDR3_DQS0_P: U1B33.IO_L21P_T3_DQS_33
- new net DDR3_DQS1_N: U1B33.IO_L15N_T2_DQS_33
- new net DDR3_DQS1_P: U1B33.IO_L15P_T2_DQS_33
- new net DDR3_DQS2_N: U1B33.IO_L9N_T1_DQS_33
- new net DDR3_DQS2_P: U1B33.IO_L9P_T1_DQS_33
- new net DDR3_DQS3_N: U1B33.IO_L3N_T0_DQS_33
- new net DDR3_DQS3_P: U1B33.IO_L3P_T0_DQS_33
- new net DDR3_ODT0: U1B34.IO_L17N_T2_34
- new net DDR3_ODT1: U1B34.IO_L18P_T2_34
- new net DDR3_RAS_B: U1B34.IO_L15N_T2_DQS_34
- new net DDR3_RESET_B: U1B34.IO_0_34
- new net DDR3_S0_B: U1B34.IO_L16N_T2_34
- new net DDR3_S1_B: U1B34.IO_L17P_T2_34
- new net DDR3_TEMP_EVENT: U1B34.IO_L18N_T2_34
- new net DDR3_WE_B: U1B34.IO_L15P_T2_DQS_34
- new net FPGA_1V5: C157.1, C158.1, U1B33.VCCO_33@0, U1B33.VCCO_33@1, U1B33.VCCO_33@2, U1B33.VCCO_33@3, U1B33.VCCO_33@4, U1B33.VCCO_33@5, U1B34.VCCO_34@0, U1B34.VCCO_34@1, U1B34.VCCO_34@2, U1B34.VCCO_34@3, U1B34.VCCO_34@4, U1B34.VCCO_34@5
- new net FPGA_3V3: C163.1, SW1.4, SW1.5, SW1.6, U1B0.CFGBVS_0, U1B0.VCCO_0@0, U1B0.VCCO_0@1
- new net FPGA_CCLK: U1B0.CCLK_0
- new net FPGA_DONE: DS10.A, J52.1, R396.2, U1B0.DONE_0
- new net FPGA_INIT_B: J52.2, U1B0.INIT_B_0
- new net FPGA_M0: R337.2, SW1.3, U1B0.M0_0
- new net FPGA_M1: R338.2, U1B0.M1_0
- new net FPGA_M2: R339.2, SW1.1, U1B0.M2_0
- new net FPGA_PROG_B: U1B0.PROGRAM_B_0
- new net FPGA_TCK_BUF: U1B0.TCK_0
- new net FPGA_TDI_BUF: U1B0.TDI_0
- new net FPGA_TMS_BUF: U1B0.TMS_0
- new net FPGA_VBATT: B1.+, R83.1, U1B0.VCCBATT_0
- new net JTAG_TDO: U1B0.TDO_0
- new net MGTAVCC: TP1A.TP, U1BMGTAVCC.MGTAVCC@0, U1BMGTAVCC.MGTAVCC@1, U1BMGTAVCC.MGTAVCC@2, U1BMGTAVCC.MGTAVCC@3, U1BMGTAVCC.MGTAVCC@4, U1BMGTAVCC.MGTAVCC@5, U1BMGTAVCC.MGTAVCC@6, U1BMGTAVCC.MGTAVCC@7, U1BMGTAVCC.MGTAVCC@8, U1BMGTAVCC.MGTAVCC@9
- new net MGTAVTT: TP2A.TP, U1BMGTAVTT.MGTAVTT@0, U1BMGTAVTT.MGTAVTT@1, U1BMGTAVTT.MGTAVTT@10, U1BMGTAVTT.MGTAVTT@11, U1BMGTAVTT.MGTAVTT@2, U1BMGTAVTT.MGTAVTT@3, U1BMGTAVTT.MGTAVTT@4, U1BMGTAVTT.MGTAVTT@5, U1BMGTAVTT.MGTAVTT@6, U1BMGTAVTT.MGTAVTT@7, U1BMGTAVTT.MGTAVTT@8, U1BMGTAVTT.MGTAVTT@9
- new net N$10: U1B33.IO_0_33
- new net N$103: U1B34.IO_L19P_T3_34
- new net N$105: U1B34.IO_L20P_T3_34
- new net N$106: U1B34.IO_L20N_T3_34
- new net N$107: U1B34.IO_L21P_T3_DQS_34
- new net N$108: U1B34.IO_L21N_T3_DQS_34
- new net N$109: U1B34.IO_L22P_T3_34
- new net N$110: U1B34.IO_L22N_T3_34
- new net N$111: U1B34.IO_L23P_T3_34
- new net N$112: U1B34.IO_L23N_T3_34
- new net N$113: U1B34.IO_L24P_T3_34
- new net N$114: U1B34.IO_L24N_T3_34
- new net N$116: U1B35.VCCO_35@0
- new net N$117: U1B35.VCCO_35@1
- new net N$118: U1B35.VCCO_35@2
- new net N$119: U1B35.VCCO_35@3
- new net N$120: U1B35.VCCO_35@4
- new net N$121: U1B35.VCCO_35@5
- new net N$122: U1B35.IO_0_35
- new net N$123: U1B35.IO_L1P_T0_AD4P_35
- new net N$124: U1B35.IO_L1N_T0_AD4N_35
- new net N$125: U1B35.IO_L2P_T0_AD12P_35
- new net N$126: U1B35.IO_L2N_T0_AD12N_35
- new net N$127: U1B35.IO_L3P_T0_DQS_AD5P_35
- new net N$128: U1B35.IO_L3N_T0_DQS_AD5N_35
- new net N$129: U1B35.IO_L4P_T0_35
- new net N$130: U1B35.IO_L4N_T0_35
- new net N$131: U1B35.IO_L5P_T0_AD13P_35
- new net N$132: U1B35.IO_L5N_T0_AD13N_35
- new net N$133: U1B35.IO_L6P_T0_35
- new net N$134: U1B35.IO_L6N_T0_VREF_35
- new net N$135: U1B35.IO_L7P_T1_AD6P_35
- new net N$136: U1B35.IO_L7N_T1_AD6N_35
- new net N$137: U1B35.IO_L8P_T1_AD14P_35
- new net N$138: U1B35.IO_L8N_T1_AD14N_35
- new net N$139: U1B35.IO_L9P_T1_DQS_AD7P_35
- new net N$140: U1B35.IO_L9N_T1_DQS_AD7N_35
- new net N$141: U1B35.IO_L10P_T1_AD15P_35
- new net N$142: U1B35.IO_L10N_T1_AD15N_35
- new net N$143: U1B35.IO_L11P_T1_SRCC_35
- new net N$144: U1B35.IO_L11N_T1_SRCC_35
- new net N$145: U1B35.IO_L12P_T1_MRCC_35
- new net N$146: U1B35.IO_L12N_T1_MRCC_35
- new net N$147: U1B35.IO_L13P_T2_MRCC_35
- new net N$148: U1B35.IO_L13N_T2_MRCC_35
- new net N$149: U1B35.IO_L14P_T2_SRCC_35
- new net N$150: U1B35.IO_L14N_T2_SRCC_35
- new net N$151: U1B35.IO_L15P_T2_DQS_35
- new net N$152: U1B35.IO_L15N_T2_DQS_35
- new net N$153: U1B35.IO_L16P_T2_35
- new net N$154: U1B35.IO_L16N_T2_35
- new net N$155: U1B35.IO_L17P_T2_35
- new net N$156: U1B35.IO_L17N_T2_35
- new net N$157: U1B35.IO_L18P_T2_35
- new net N$158: U1B35.IO_L18N_T2_35
- new net N$159: U1B35.IO_L19P_T3_35
- new net N$160: U1B35.IO_L19N_T3_VREF_35
- new net N$161: U1B35.IO_L20P_T3_35
- new net N$162: U1B35.IO_L20N_T3_35
- new net N$163: U1B35.IO_L21P_T3_DQS_35
- new net N$164: U1B35.IO_L21N_T3_DQS_35
- new net N$165: U1B35.IO_L22P_T3_35
- new net N$166: U1B35.IO_L22N_T3_35
- new net N$167: U1B35.IO_L23P_T3_35
- new net N$168: U1B35.IO_L23N_T3_35
- new net N$169: U1B35.IO_L24P_T3_35
- new net N$170: U1B35.IO_L24N_T3_35
- new net N$171: U1B35.IO_25_35
- new net N$34: U1B33.IO_L12N_T1_MRCC_33
- new net N$4: U1BTDIODE.DXP_0
- new net N$46: U1B33.IO_L18N_T2_33
- new net N$5: U1BTDIODE.DXN_0
- new net N$59: U1B33.IO_25_33
- new net N$6: D6.A1, R83.2
- new net SYSCLK_N: U1B34.IO_L13N_T2_MRCC_34
- new net SYSCLK_P: U1B34.IO_L13P_T2_MRCC_34
- new net VCC1V8: D6.C2
- new net VCCAUX: U1BVCCAUX.VCCAUX@0, U1BVCCAUX.VCCAUX@1, U1BVCCAUX.VCCAUX@2, U1BVCCAUX.VCCAUX@3, U1BVCCAUX.VCCAUX@4
- new net VCCBRAM: U1BVCCBRAM.VCCBRAM@0, U1BVCCBRAM.VCCBRAM@1, U1BVCCBRAM.VCCBRAM@2, U1BVCCBRAM.VCCBRAM@3
- new net VCCINT: U1BVCCINT.VCCINT@0, U1BVCCINT.VCCINT@1, U1BVCCINT.VCCINT@10, U1BVCCINT.VCCINT@11, U1BVCCINT.VCCINT@12, U1BVCCINT.VCCINT@2, U1BVCCINT.VCCINT@3, U1BVCCINT.VCCINT@4, U1BVCCINT.VCCINT@5, U1BVCCINT.VCCINT@6, U1BVCCINT.VCCINT@7, U1BVCCINT.VCCINT@8, U1BVCCINT.VCCINT@9
- new net XADC_AGND: C1.2, C2.2, U1BXADC.GNDADC_0, U1BXADC.VREFN_0
- new net XADC_VCC: C2.1, U1BXADC.VCCADC_0
- new net XADC_VN_R_N: U1BXADC.VN_0
- new net XADC_VP_R_P: U1BXADC.VP_0
- new net XADC_VREFP: C1.1, U1BXADC.VREFP_0
- net GND: now also B1.-, C157.2, C158.2, C163.2, C461.2, C462.2, C490.2, C491.2, DS10.C, R337.1, R338.1, R339.1, TP1B.TP, TP2B.TP, U1BGNDA.GND@0, U1BGNDA.GND@1, U1BGNDA.GND@10, U1BGNDA.GND@11, U1BGNDA.GND@12, U1BGNDA.GND@13, U1BGNDA.GND@14, U1BGNDA.GND@15, U1BGNDA.GND@16, U1BGNDA.GND@17, U1BGNDA.GND@18, U1BGNDA.GND@19, U1BGNDA.GND@2, U1BGNDA.GND@20, U1BGNDA.GND@21, U1BGNDA.GND@22, U1BGNDA.GND@23, U1BGNDA.GND@24, U1BGNDA.GND@25, U1BGNDA.GND@26, U1BGNDA.GND@27, U1BGNDA.GND@28, U1BGNDA.GND@29, U1BGNDA.GND@3, U1BGNDA.GND@30, U1BGNDA.GND@31, U1BGNDA.GND@32, U1BGNDA.GND@33, U1BGNDA.GND@34, U1BGNDA.GND@35, U1BGNDA.GND@36, U1BGNDA.GND@37, U1BGNDA.GND@38, U1BGNDA.GND@39, U1BGNDA.GND@4, U1BGNDA.GND@5, U1BGNDA.GND@6, U1BGNDA.GND@7, U1BGNDA.GND@8, U1BGNDA.GND@9, U1BGNDB.GND@40, U1BGNDB.GND@41, U1BGNDB.GND@42, U1BGNDB.GND@43, U1BGNDB.GND@44, U1BGNDB.GND@45, U1BGNDB.GND@46, U1BGNDB.GND@47, U1BGNDB.GND@48, U1BGNDB.GND@49, U1BGNDB.GND@50, U1BGNDB.GND@51, U1BGNDB.GND@52, U1BGNDB.GND@53, U1BGNDB.GND@54, U1BGNDB.GND@55, U1BGNDB.GND@56, U1BGNDB.GND@57, U1BGNDB.GND@58, U1BGNDB.GND@59, U1BGNDB.GND@60, U1BGNDB.GND@61, U1BGNDB.GND@62, U1BGNDB.GND@63, U1BGNDB.GND@64, U1BGNDB.GND@65, U1BGNDB.GND@66, U1BGNDB.GND@67, U1BGNDB.GND@68, U1BGNDB.GND@69, U1BGNDB.GND@70, U1BGNDB.GND@71, U1BGNDB.GND@72, U1BGNDB.GND@73, U1BGNDB.GND@74, U1BGNDB.GND@75, U1BGNDB.GND@76, U1BGNDB.GND@77, U1BGNDB.GND@78, U1BGNDB.GND@79, U1BGNDC.GND@100, U1BGNDC.GND@101, U1BGNDC.GND@102, U1BGNDC.GND@103, U1BGNDC.GND@104, U1BGNDC.GND@105, U1BGNDC.GND@106, U1BGNDC.GND@107, U1BGNDC.GND@108, U1BGNDC.GND@109, U1BGNDC.GND@110, U1BGNDC.GND@111, U1BGNDC.GND@112, U1BGNDC.GND@113, U1BGNDC.GND@114, U1BGNDC.GND@115, U1BGNDC.GND@116, U1BGNDC.GND@117, U1BGNDC.GND@118, U1BGNDC.GND@80, U1BGNDC.GND@81, U1BGNDC.GND@82, U1BGNDC.GND@83, U1BGNDC.GND@84, U1BGNDC.GND@85, U1BGNDC.GND@86, U1BGNDC.GND@87, U1BGNDC.GND@88, U1BGNDC.GND@89, U1BGNDC.GND@90, U1BGNDC.GND@91, U1BGNDC.GND@92, U1BGNDC.GND@93, U1BGNDC.GND@94, U1BGNDC.GND@95, U1BGNDC.GND@96, U1BGNDC.GND@97, U1BGNDC.GND@98, U1BGNDC.GND@99; no longer J1.197, J1.198, J1.201, U2BGNDA.GND@0, U2BGNDA.GND@1, U2BGNDA.GND@10, U2BGNDA.GND@11, U2BGNDA.GND@12, U2BGNDA.GND@13, U2BGNDA.GND@14, U2BGNDA.GND@15, U2BGNDA.GND@16, U2BGNDA.GND@17, U2BGNDA.GND@18, U2BGNDA.GND@19, U2BGNDA.GND@2, U2BGNDA.GND@20, U2BGNDA.GND@21, U2BGNDA.GND@22, U2BGNDA.GND@23, U2BGNDA.GND@24, U2BGNDA.GND@25, U2BGNDA.GND@26, U2BGNDA.GND@27, U2BGNDA.GND@28, U2BGNDA.GND@29, U2BGNDA.GND@3, U2BGNDA.GND@30, U2BGNDA.GND@31, U2BGNDA.GND@32, U2BGNDA.GND@33, U2BGNDA.GND@34, U2BGNDA.GND@35, U2BGNDA.GND@36, U2BGNDA.GND@37, U2BGNDA.GND@38, U2BGNDA.GND@39, U2BGNDA.GND@4, U2BGNDA.GND@5, U2BGNDA.GND@6, U2BGNDA.GND@7, U2BGNDA.GND@8, U2BGNDA.GND@9, U2BGNDB.GND@40, U2BGNDB.GND@41, U2BGNDB.GND@42, U2BGNDB.GND@43, U2BGNDB.GND@44, U2BGNDB.GND@45, U2BGNDB.GND@46, U2BGNDB.GND@47, U2BGNDB.GND@48, U2BGNDB.GND@49, U2BGNDB.GND@50, U2BGNDB.GND@51, U2BGNDB.GND@52, U2BGNDB.GND@53, U2BGNDB.GND@54, U2BGNDB.GND@55, U2BGNDB.GND@56, U2BGNDB.GND@57, U2BGNDB.GND@58, U2BGNDB.GND@59, U2BGNDB.GND@60, U2BGNDB.GND@61, U2BGNDB.GND@62, U2BGNDB.GND@63, U2BGNDB.GND@64, U2BGNDB.GND@65, U2BGNDB.GND@66, U2BGNDB.GND@67, U2BGNDB.GND@68, U2BGNDB.GND@69, U2BGNDB.GND@70, U2BGNDB.GND@71, U2BGNDB.GND@72, U2BGNDB.GND@73, U2BGNDB.GND@74, U2BGNDB.GND@75, U2BGNDB.GND@76, U2BGNDB.GND@77, U2BGNDB.GND@78, U2BGNDB.GND@79, U2BGNDC.GND@100, U2BGNDC.GND@101, U2BGNDC.GND@102, U2BGNDC.GND@103, U2BGNDC.GND@104, U2BGNDC.GND@105, U2BGNDC.GND@106, U2BGNDC.GND@107, U2BGNDC.GND@108, U2BGNDC.GND@109, U2BGNDC.GND@110, U2BGNDC.GND@111, U2BGNDC.GND@112, U2BGNDC.GND@113, U2BGNDC.GND@114, U2BGNDC.GND@115, U2BGNDC.GND@116, U2BGNDC.GND@117, U2BGNDC.GND@118, U2BGNDC.GND@119, U2BGNDC.GND@80, U2BGNDC.GND@81, U2BGNDC.GND@82, U2BGNDC.GND@83, U2BGNDC.GND@84, U2BGNDC.GND@85, U2BGNDC.GND@86, U2BGNDC.GND@87, U2BGNDC.GND@88, U2BGNDC.GND@89, U2BGNDC.GND@90, U2BGNDC.GND@91, U2BGNDC.GND@92, U2BGNDC.GND@93, U2BGNDC.GND@94, U2BGNDC.GND@95, U2BGNDC.GND@96, U2BGNDC.GND@97, U2BGNDC.GND@98, U2BGNDC.GND@99
- net VCC3V3: now also R396.1; no longer J1.199
- net VTTVREF: now also C461.1, C462.1, C490.1, C491.1, U1B33.IO_L19N_T3_VREF_33, U1B33.IO_L6N_T0_VREF_33, U1B34.IO_L19N_T3_VREF_34, U1B34.IO_L6N_T0_VREF_34; no longer J1.1, J1.124, J1.126
Other:
- note removed: "A0"
- note removed: "A1"
- note removed: "A10"
- note removed: "A11"
- note removed: "A12"
- note removed: "A13"
- note removed: "A14"
- note removed: "A15"
- note removed: "A2"
- note removed: "A3"
- note removed: "A4"
- note removed: "A5"
- note removed: "A6"
- note removed: "A7"
- note removed: "A8"
- note removed: "A9"
- note removed: "BA0"
- note removed: "BA1"
- note removed: "BA2"
- note removed: "CAS#"
- note removed: "CK0"
- note removed: "CK0#"
- note removed: "CK1"
- note removed: "CK1#"
- note removed: "CKE0"
- note removed: "DM0"
- note removed: "DM1"
- note removed: "DM2"
- note removed: "DM3"
- note removed: "DM4"
- note removed: "DM5"
- note removed: "DM6"
- note removed: "DM7"
- note removed: "DQ0"
- note removed: "DQ1"
- note removed: "DQ10"
- note removed: "DQ11"
- note removed: "DQ12"
- note removed: "DQ13"
- note removed: "DQ14"
- note removed: "DQ15"
- note removed: "DQ16"
- note removed: "DQ17"
- note removed: "DQ18"
- note removed: "DQ19"
- note removed: "DQ2"
- note removed: "DQ20"
- note removed: "DQ21"
- note removed: "DQ22"
- note removed: "DQ23"
- note removed: "DQ24"
- note removed: "DQ25"
- note removed: "DQ26"
- note removed: "DQ27"
- note removed: "DQ28"
- note removed: "DQ29"
- note removed: "DQ3"
- note removed: "DQ3#"
- note removed: "DQ30"
- note removed: "DQ31"
- note removed: "DQ32"
- note removed: "DQ33"
- note removed: "DQ34"
- note removed: "DQ35"
- note removed: "DQ36"
- note removed: "DQ37"
- note removed: "DQ38"
- note removed: "DQ39"
- note removed: "DQ4"
- note removed: "DQ40"
- note removed: "DQ41"
- note removed: "DQ42"
- note removed: "DQ43"
- note removed: "DQ44"
- note removed: "DQ45"
- note removed: "DQ46"
- note removed: "DQ47"
- note removed: "DQ48"
- note removed: "DQ49"
- note removed: "DQ5"
- note removed: "DQ50"
- note removed: "DQ51"
- note removed: "DQ52"
- note removed: "DQ53"
- note removed: "DQ54"
- note removed: "DQ55"
- note removed: "DQ56"
- note removed: "DQ57"
- note removed: "DQ58"
- note removed: "DQ59"
- note removed: "DQ6"
- note removed: "DQ60"
- note removed: "DQ61"
- note removed: "DQ62"
- note removed: "DQ63"
- note removed: "DQ7"
- note removed: "DQ8"
- note removed: "DQ9"
- note removed: "DQS0"
- note removed: "DQS0#"
- note removed: "DQS1"
- note removed: "DQS1#"
- note removed: "DQS2"
- note removed: "DQS2#"
- note removed: "DQS4"
- note removed: "DQS4#"
- note removed: "DQS5"
- note removed: "DQS5#"
- note removed: "DQS6"
- note removed: "DQS6#"
- note removed: "DQS7"
- note removed: "DQS7#"
- note removed: "NC"
- note removed: "NF"
- note removed: "ODT0"
- note removed: "RAS#"
- note removed: "RESET"
- note removed: "S0#"
- note removed: "SA0"
- note removed: "SA1"
- note removed: "SCL"
- note removed: "SDA"
- note removed: "Vdd"
- note removed: "Vddspd"
- note removed: "Vrefca"
- note removed: "Vrefdq"
- note removed: "Vss"
- note removed: "Vtt"
- note removed: "WE#"

Commit message: adding 35
Parts:
- added C402: 100UF, eagle-ltspice:CC1206
- added C463, C492: 0.1UF, eagle-ltspice:CC0402
Connections:
- net N$123 renamed DDR3_D63
- net N$124 renamed DDR3_D62
- net N$125 renamed DDR3_D61
- net N$126 renamed DDR3_D60
- net N$127 renamed DDR3_DQS7_P
- net N$128 renamed DDR3_DQS7_N
- net N$129 renamed DDR3_D59
- net N$130 renamed DDR3_D58
- net N$131 renamed DDR3_D57
- net N$132 renamed DDR3_D56
- net N$133 renamed DDR3_DM7
- net N$135 renamed DDR3_D55
- net N$136 renamed DDR3_D54
- net N$137 renamed DDR3_D53
- net N$138 renamed DDR3_D52
- net N$139 renamed DDR3_DQS6_P
- net N$140 renamed DDR3_DQS6_N
- net N$141 renamed DDR3_D51
- net N$142 renamed DDR3_D50
- net N$143 renamed DDR3_D49
- net N$144 renamed DDR3_D48
- net N$145 renamed DDR3_DM6
- net N$147 renamed DDR3_D47
- net N$148 renamed DDR3_D46
- net N$149 renamed DDR3_D45
- net N$150 renamed DDR3_D44
- net N$151 renamed DDR3_DQS5_P
- net N$152 renamed DDR3_DQS5_N
- net N$153 renamed DDR3_D43
- net N$154 renamed DDR3_D42
- net N$155 renamed DDR3_D41
- net N$156 renamed DDR3_D40
- net N$157 renamed DDR3_DM5
- net N$159 renamed DDR3_D39
- net N$161 renamed DDR3_D38
- net N$162 renamed DDR3_D37
- net N$163 renamed DDR3_DQS4_P
- net N$164 renamed DDR3_DQS4_N
- net N$165 renamed DDR3_D36
- net N$166 renamed DDR3_D35
- net N$167 renamed DDR3_D34
- net N$168 renamed DDR3_D33
- net N$169 renamed DDR3_D32
- net N$170 renamed DDR3_DM4
- removed net N$119: U1B35.VCCO_35@3
- removed net N$134: U1B35.IO_L6N_T0_VREF_35
- removed net N$160: U1B35.IO_L19N_T3_VREF_35
- net FPGA_1V5: now also C402.1, U1B35.VCCO_35@3
- net GND: now also C402.2, C463.2, C492.2
- net VTTVREF: now also C463.1, C492.1, U1B35.IO_L19N_T3_VREF_35, U1B35.IO_L6N_T0_VREF_35
Other:
- moved on the sheet: U1B35
